File: misc/misc.kicad_sch (KiCad schematic)
At the start: 4 parts, among them SW1 SW_SPST

Commit message: update
Parts:
- added M1: Motor_DC, symbol Motor:Motor_DC
- added Q1: IRLB4132, symbol Simulation_SPICE:NMOS
- added R1: 10K, symbol Device:R_US
- added R2: 1K, symbol Device:R_US
- added U4: LD1117V33, Package_TO_SOT_SMD:SOT-223-3_TabPin2, symbol Regulator_Linear:LD1117S33TR_SOT223
Connections:
- new net: Q1.2 (G), R1.1, R2.2
- new net: M1.1 (+), U4.2 (VO)
- new net: M1.2 (-), Q1.1 (D)
- new net GND: Q1.3 (S), R1.2, U4.1 (GND)
Other:
- note added: "+3.3V from Teensy digital out pin"
- note added: "+5V from power reg. (Pololu)"
Changed lines of the file:
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@@
 (kicad_sch (version 20230121) (generator eeschema)
   (paper "A4")
+  (junction (at 49.53 154.94) (diameter 0) (color 0 0 0 0)
+  )
   (no_connect (at 129.54 88.9))
   (no_connect (at 135.89 99.06))
@@
     (stroke (width 0) (type default))
   )
+  (wire (pts (xy 62.23 162.56) (xy 62.23 160.02))
+    (stroke (width 0) (type default))
+  )
+  (wire (pts (xy 49.53 154.94) (xy 54.61 154.94))
+    (stroke (width 0) (type default))
+  )
+  (wire (pts (xy 62.23 137.16) (xy 62.23 135.89))
+    (stroke (width 0) (type default))
+  )
+  (wire (pts (xy 36.83 135.89) (xy 41.91 135.89))
+    (stroke (width 0) (type default))
+  )
   (wire (pts (xy 149.86 115.57) (xy 149.86 125.73))
     (stroke (width 0) (type default))
@@
     (stroke (width 0) (type default))
   )
+  (wire (pts (xy 57.15 135.89) (xy 62.23 135.89))
+    (stroke (width 0) (type default))
+  )
   (wire (pts (xy 152.4 115.57) (xy 152.4 128.27))
     (stroke (width 0) (type default))
   )
+  (wire (pts (xy 36.83 154.94) (xy 41.91 154.94))
+    (stroke (width 0) (type default))
+  )
   (wire (pts (xy 142.24 128.27) (xy 152.4 128.27))
     (stroke (width 0) (type default))
@@
     (stroke (width 0) (type default))
   )
+  (text "+5V from \npower reg.\n(Pololu)\n" (at 25.4 138.43 0)
+    (effects (font (size 1.27 1.27)) (justify left bottom))
+  )
+  (text "+3.3V from \nTeensy digital\nout pin\n" (at 25.4 156.21 0)
+    (effects (font (size 1.27 1.27)) (justify left bottom))
+  )
+  (symbol (lib_id "Device:R_US") (at 45.72 154.94 90) (unit 1)
+    (in_bom yes) (on_board yes) (dnp no)
+    (property "Reference" "R2" (at 44.45 152.4 90)
+      (effects (font (size 1.27 1.27)) (justify right))
+    )
+    (property "Value" "1K" (at 46.99 152.4 90) (do_not_autoplace)
+      (effects (font (size 1.27 1.27)) (justify right bottom))
+    )
+    (property "Footprint" "" (at 45.974 153.924 90)
+      (effects (font (size 1.27 1.27)) hide)
+    )
+    (property "Datasheet" "~" (at 45.72 154.94 0)
+      (effects (font (size 1.27 1.27)) hide)
+    )
+    (pin "1")
+    (pin "2")
+    (instances
+      (project "misc"
+        (path "/c4ef71c4-9905-4c9e-8a7f-b12eb68ee77a"
+          (reference "R2") (unit 1)
+        )
+      )
+    )
+  )
+  (symbol (lib_id "Motor:Motor_DC") (at 62.23 142.24 0) (unit 1)
+    (in_bom yes) (on_board yes) (dnp no) (fields_autoplaced)
+    (property "Reference" "M1" (at 67.31 143.51 0)
+      (effects (font (size 1.27 1.27)) (justify left))
+    )
+    (property "Value" "Motor_DC" (at 67.31 146.05 0)
+      (effects (font (size 1.27 1.27)) (justify left))
+    )
+    (property "Footprint" "" (at 62.23 144.526 0)
+      (effects (font (size 1.27 1.27)) hide)
+    )
+    (property "Datasheet" "~" (at 62.23 144.526 0)
+      (effects (font (size 1.27 1.27)) hide)
+    )
+    (pin "1")
+    (pin "2")
+    (instances
+      (project "misc"
+        (path "/c4ef71c4-9905-4c9e-8a7f-b12eb68ee77a"
+          (reference "M1") (unit 1)
+        )
+      )
+    )
+  )
   (symbol (lib_id "Jstconnector:jstcon") (at 124.46 121.92 0) (unit 1)
     (in_bom yes) (on_board yes) (dnp no) (fields_autoplaced)
@@
         (path "/c4ef71c4-9905-4c9e-8a7f-b12eb68ee77a"
           (reference "SW1") (unit 1)
+        )
+      )
+    )
+  )
+  (symbol (lib_id "power:GND") (at 49.53 143.51 0) (unit 1)
+    (in_bom yes) (on_board yes) (dnp no) (fields_autoplaced)
+    (property "Reference" "#PWR01" (at 49.53 149.86 0)
+      (effects (font (size 1.27 1.27)) hide)
+    )
+    (property "Value" "GND" (at 49.53 148.59 0)
+      (effects (font (size 1.27 1.27)))
+    )
+    (property "Footprint" "" (at 49.53 143.51 0)
+      (effects (font (size 1.27 1.27)) hide)
+    )
+    (property "Datasheet" "" (at 49.53 143.51 0)
+      (effects (font (size 1.27 1.27)) hide)
+    )
+    (pin "1")
+    (instances
+      (project "misc"
+        (path "/c4ef71c4-9905-4c9e-8a7f-b12eb68ee77a"
+          (reference "#PWR01") (unit 1)
+        )
+      )
+    )
+  )
+  (symbol (lib_id "Regulator_Linear:LD1117S33TR_SOT223") (at 49.53 135.89 0) (unit 1)
+    (in_bom yes) (on_board yes) (dnp no) (fields_autoplaced)
+    (property "Reference" "U4" (at 49.53 129.54 0)
+      (effects (font (size 1.27 1.27)))
+    )
+    (property "Value" "LD1117V33 " (at 49.53 132.08 0)
+      (effects (font (size 1.27 1.27)))
+    )
+    (property "Footprint" "Package_TO_SOT_SMD:SOT-223-3_TabPin2" (at 49.53 130.81 0)
+      (effects (font (size 1.27 1.27)) hide)
+    )
+    (property "Datasheet" "http://www.st.com/st-web-ui/static/active/en/resource/technical/document/datasheet/CD00000544.pdf" (at 52.07 142.24 0)
+      (effects (font (size 1.27 1.27)) hide)
+    )
+    (pin "3")
+    (pin "1")
+    (pin "2")
+    (instances
+      (project "misc"
+        (path "/c4ef71c4-9905-4c9e-8a7f-b12eb68ee77a"
+          (reference "U4") (unit 1)
+        )
+      )
+    )
+  )
+  (symbol (lib_id "power:GND") (at 62.23 162.56 0) (unit 1)
+    (in_bom yes) (on_board yes) (dnp no) (fields_autoplaced)
+    (property "Reference" "#PWR02" (at 62.23 168.91 0)
+      (effects (font (size 1.27 1.27)) hide)
+    )
+    (property "Value" "GND" (at 62.23 167.64 0)
+      (effects (font (size 1.27 1.27)))
+    )
+    (property "Footprint" "" (at 62.23 162.56 0)
+      (effects (font (size 1.27 1.27)) hide)
+    )
+    (property "Datasheet" "" (at 62.23 162.56 0)
+      (effects (font (size 1.27 1.27)) hide)
+    )
+    (pin "1")
+    (instances
+      (project "misc"
+        (path "/c4ef71c4-9905-4c9e-8a7f-b12eb68ee77a"
+          (reference "#PWR02") (unit 1)
         )
       )
@@
         )
       )
+    )
+  )
+  (symbol (lib_id "power:GND") (at 49.53 162.56 0) (unit 1)
+    (in_bom yes) (on_board yes) (dnp no) (fields_autoplaced)
+    (property "Reference" "#PWR03" (at 49.53 168.91 0)
+      (effects (font (size 1.27 1.27)) hide)
+    )
+    (property "Value" "GND" (at 49.53 167.64 0)
+      (effects (font (size 1.27 1.27)))
+    )
+    (property "Footprint" "" (at 49.53 162.56 0)
+      (effects (font (size 1.27 1.27)) hide)
+    )
+    (property "Datasheet" "" (at 49.53 162.56 0)
+      (effects (font (size 1.27 1.27)) hide)
+    )
+    (pin "1")
+    (instances
+      (project "misc"
+        (path "/c4ef71c4-9905-4c9e-8a7f-b12eb68ee77a"
+          (reference "#PWR03") (unit 1)
+        )
+      )
+    )
+  )
+  (symbol (lib_id "Device:R_US") (at 49.53 158.75 0) (unit 1)
+    (in_bom yes) (on_board yes) (dnp no)
+    (property "Reference" "R1" (at 52.07 157.48 0)
+      (effects (font (size 1.27 1.27)) (justify left))
+    )
+    (property "Value" "10K" (at 52.07 160.02 0) (do_not_autoplace)
+      (effects (font (size 1.27 1.27)) (justify left top))
+    )
+    (property "Footprint" "" (at 50.546 159.004 90)
+      (effects (font (size 1.27 1.27)) hide)
+    )
+    (property "Datasheet" "~" (at 49.53 158.75 0)
+      (effects (font (size 1.27 1.27)) hide)
+    )
+    (pin "1")
+    (pin "2")
+    (instances
+      (project "misc"
+        (path "/c4ef71c4-9905-4c9e-8a7f-b12eb68ee77a"
+          (reference "R1") (unit 1)
+        )
+      )
+    )
+  )
+  (symbol (lib_id "Simulation_SPICE:NMOS") (at 59.69 154.94 0) (unit 1)
+    (in_bom yes) (on_board yes) (dnp no) (fields_autoplaced)
+    (property "Reference" "Q1" (at 66.04 153.67 0)
+      (effects (font (size 1.27 1.27)) (justify left))
+    )
+    (property "Value" "IRLB4132" (at 66.04 156.21 0)
+      (effects (font (size 1.27 1.27)) (justify left))
+    )
+    (property "Footprint" "" (at 64.77 152.4 0)
+      (effects (font (size 1.27 1.27)) hide)
+    )
+    (property "Datasheet" "https://ngspice.sourceforge.io/docs/ngspice-manual.pdf" (at 59.69 167.64 0)
+      (effects (font (size 1.27 1.27)) hide)
+    )
+    (property "Sim.Device" "NMOS" (at 59.69 172.085 0)
+      (effects (font (size 1.27 1.27)) hide)
+    )
+    (property "Sim.Type" "VDMOS" (at 59.69 173.99 0)
+      (effects (font (size 1.27 1.27)) hide)
+    )
+    (property "Sim.Pins" "1=D 2=G 3=S" (at 59.69 170.18 0)
+      (effects (font (size 1.27 1.27)) hide)
+    )
+    (pin "1")
+    (pin "3")
+    (pin "2")
+    (instances
+      (project "misc"
+        (path "/c4ef71c4-9905-4c9e-8a7f-b12eb68ee77a"
+          (reference "Q1") (unit 1)
+        )
+      )
