File: payload24.kicad_pcb (KiCad board)
At the start: 6 copper layers, 81.9 x 89.4 mm, 20 parts, among them J1 JST-XH3, J2 PixHawk, J3 Motors, J4 Motors, Q2 CSD19503KCS, Q3 IRLB4132, SW1 FingerTech, U2 LMS1585ACT-3.3/NOPB, U7 LMS1585ACT-3.3/NOPB

Commit message: update
Parts:
- added C1: 10μF, CAPC3216X110N:CAPC3216X110N, B.Cu at (86.6, 73.4)
- added C2: 10μF, CAPC3216X110N:CAPC3216X110N, B.Cu at (86.5, 77.0)
- added C3: 10μF, CAPC3216X110N:CAPC3216X110N, B.Cu at (86.5, 80.7)
Other:
- outline, holes or cut-outs redrawn
- board text added: "10μ"
